File: Documents/EagleSchematics/HC16_SENSOR_NOMUX/STRAIGT_SENSOR_NOMUX_16.brd (EAGLE design)
At the start: 298.1 x 33.6 mm, 33 parts

Commit message: Eagle Schematics
Changed array of sensornetwork
Parts:
- removed R1, R10, R11, R12, R13, R14, R15, R16, R2, R3, R4, R5, R6, R7, R8, R9: 10k, resistor:0207/10
- added IR, IR1, IR10, IR11, IR12, IR13, IR14, IR2, IR3, IR4, IR5, IR6, IR7, IR8, IR9: SFH482, led:SFH482
- added R17, R18, R19, R20, R21, R22, R23, R24, R25, R26, R27, R28, R29, R30, R31: 100, resistor:0207/10
Connections:
- new net N$1: IR1.A, R18.1
- new net N$10: IR9.A, R26.1
- new net N$11: IR10.A, R27.1
- new net N$12: IR11.A, R28.1
- new net N$13: IR12.A, R29.1
- new net N$14: IR13.A, R30.1
- new net N$15: IR14.A, R31.1
- new net N$2: IR.A, R17.1
- new net N$3: IR2.A, R19.1
- new net N$4: IR3.A, R20.1
- new net N$5: IR4.A, R21.1
- new net N$6: IR5.A, R22.1
- new net N$7: IR6.A, R23.1
- new net N$8: IR7.A, R24.1
- new net N$9: IR8.A, R25.1
- net +3V3: now also R17.2, R18.2, R19.2, R20.2, R21.2, R22.2, R23.2, R24.2, R25.2, R26.2, R27.2, R28.2, R29.2, R30.2, R31.2
- net GND: now also IR.K, IR1.K, IR10.K, IR11.K, IR12.K, IR13.K, IR14.K, IR2.K, IR3.K, IR4.K, IR5.K, IR6.K, IR7.K, IR8.K, IR9.K; no longer R1.2, R10.2, R11.2, R12.2, R13.2, R14.2, R15.2, R16.2, R2.2, R3.2, R4.2, R5.2, R6.2, R7.2, R8.2, R9.2
- net PHOTO1: no longer R8.1
- net PHOTO10: no longer R10.1
- net PHOTO11: no longer R11.1
- net PHOTO12: no longer R12.1
- net PHOTO13: no longer R13.1
- net PHOTO14: no longer R14.1
- net PHOTO15: no longer R15.1
- net PHOTO16: no longer R16.1
- net PHOTO2: no longer R7.1
- net PHOTO3: no longer R6.1
- net PHOTO4: no longer R5.1
- net PHOTO5: no longer R4.1
- net PHOTO6: no longer R3.1
- net PHOTO7: no longer R2.1
- net PHOTO8: no longer R1.1
- net PHOTO9: no longer R9.1
Routing:
- net PHOTO8: track 5.08 -> 0.00 mm
- net PHOTO6: track 5.08 -> 0.00 mm
- net PHOTO5: track 5.08 -> 0.00 mm
- net PHOTO4: track 5.08 -> 0.00 mm
- net PHOTO3: track 5.08 -> 0.00 mm
- net PHOTO2: track 5.08 -> 0.00 mm
- net PHOTO1: track 5.08 -> 0.00 mm

Commit message: Almost final version of schematics
Updated BigBoard with the new design
Parts:
- moved 20X_SENSOR 10.5 mm to (195.6, 0.00), turned to 180 degrees
- moved R17 5.08 mm to (10.2, 22.9)
Connections:
- new net +5V: 20X_SENSOR.2
- net +3V3: no longer 20X_SENSOR.2
Changed lines of the file:
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@@
 <attribute name="NAME" x="237.1950625" y="10.454934375" size="1.27" layer="25" ratio="10" rot="R315"/>
 </element>
-<element name="20X_SENSOR" library="Wuerth_Elektronik_eiCan_05_Box_Header_IDC_Connectors_1_2" package="61202022021" value="61202022021" x="205.74" y="-2.54"/>
-<element name="R17" library="resistor" package="0207/10" value="100" x="10.16" y="17.78" rot="R180"/>
+<element name="20X_SENSOR" library="Wuerth_Elektronik_eiCan_05_Box_Header_IDC_Connectors_1_2" package="61202022021" value="61202022021" x="195.58" y="0" rot="R180"/>
+<element name="R17" library="resistor" package="0207/10" value="100" x="10.16" y="22.86" rot="R180"/>
 <element name="IR" library="led" package="SFH482" value="SFH482" x="13.97" y="15.113"/>
 <element name="R18" library="resistor" package="0207/10" value="100" x="25.4" y="17.78" rot="R180"/>
@@
 <wire x1="30.48" y1="15.24" x2="45.593" y2="15.113" width="0" layer="19" extent="1-1"/>
 <wire x1="15.24" y1="15.113" x2="30.48" y2="15.24" width="0" layer="19" extent="1-1"/>
-<wire x1="210.82" y1="-1.27" x2="213.233" y2="15.113" width="0" layer="19" extent="1-1"/>
+<wire x1="190.5" y1="-1.27" x2="121.92" y2="15.24" width="0" layer="19" extent="1-1"/>
 </signal>
 <signal name="+3V3">
@@
 <contactref element="D15" pad="A"/>
 <contactref element="D16" pad="A"/>
-<contactref element="20X_SENSOR" pad="2"/>
 <contactref element="R17" pad="2"/>
 <contactref element="R18" pad="2"/>
@@
 <wire x1="20.32" y1="17.78" x2="35.56" y2="17.78" width="0" layer="19" extent="1-1"/>
 <wire x1="20.3327625" y1="12.7" x2="20.32" y2="17.78" width="0" layer="19" extent="1-1"/>
-<wire x1="5.08" y1="17.78" x2="20.32" y2="17.78" width="0" layer="19" extent="1-1"/>
-<wire x1="5.0927625" y1="12.7" x2="5.08" y2="17.78" width="0" layer="19" extent="1-1"/>
-<wire x1="210.82" y1="-3.81" x2="218.4527625" y2="12.7" width="0" layer="19" extent="1-1"/>
+<wire x1="5.08" y1="22.86" x2="20.32" y2="17.78" width="0" layer="19" extent="1-1"/>
+<wire x1="5.0927625" y1="12.7" x2="5.08" y2="22.86" width="0" layer="19" extent="1-1"/>
 </signal>
 <signal name="PHOTO16">
 <contactref element="D16" pad="K"/>
 <contactref element="20X_SENSOR" pad="18"/>
-<wire x1="190.5" y1="-3.81" x2="236.207234375" y2="12.7" width="0" layer="19" extent="1-1"/>
+<wire x1="210.82" y1="1.27" x2="236.207234375" y2="12.7" width="0" layer="19" extent="1-1"/>
 </signal>
 <signal name="PHOTO1">
 <contactref element="D8" pad="K"/>
 <contactref element="20X_SENSOR" pad="3"/>
-<wire x1="114.287234375" y1="12.7" x2="208.28" y2="-1.27" width="0" layer="19" extent="1-1"/>
+<wire x1="193.04" y1="-1.27" x2="114.287234375" y2="12.7" width="0" layer="19" extent="1-1"/>
 </signal>
 <signal name="PHOTO2">
 <contactref element="D7" pad="K"/>
 <contactref element="20X_SENSOR" pad="5"/>
-<wire x1="99.047234375" y1="12.7" x2="205.74" y2="-1.27" width="0" layer="19" extent="1-1"/>
+<wire x1="195.58" y1="-1.27" x2="99.047234375" y2="12.7" width="0" layer="19" extent="1-1"/>
 </signal>
 <signal name="PHOTO3">
 <contactref element="D6" pad="K"/>
 <contactref element="20X_SENSOR" pad="7"/>
-<wire x1="83.807234375" y1="12.7" x2="203.2" y2="-1.27" width="0" layer="19" extent="1-1"/>
+<wire x1="198.12" y1="-1.27" x2="83.807234375" y2="12.7" width="0" layer="19" extent="1-1"/>
 </signal>
 <signal name="PHOTO4">
@@
 <contactref element="D4" pad="K"/>
 <contactref element="20X_SENSOR" pad="11"/>
-<wire x1="53.327234375" y1="12.7" x2="198.12" y2="-1.27" width="0" layer="19" extent="1-1"/>
+<wire x1="53.327234375" y1="12.7" x2="203.2" y2="-1.27" width="0" layer="19" extent="1-1"/>
 </signal>
 <signal name="PHOTO6">
 <contactref element="D3" pad="K"/>
 <contactref element="20X_SENSOR" pad="13"/>
-<wire x1="38.087234375" y1="12.7" x2="195.58" y2="-1.27" width="0" layer="19" extent="1-1"/>
+<wire x1="38.087234375" y1="12.7" x2="205.74" y2="-1.27" width="0" layer="19" extent="1-1"/>
 </signal>
 <signal name="PHOTO7">
 <contactref element="D2" pad="K"/>
 <contactref element="20X_SENSOR" pad="15"/>
-<wire x1="22.847234375" y1="12.7" x2="193.04" y2="-1.27" width="0" layer="19" extent="1-1"/>
+<wire x1="22.847234375" y1="12.7" x2="208.28" y2="-1.27" width="0" layer="19" extent="1-1"/>
 </signal>
 <signal name="PHOTO8">
 <contactref element="D1" pad="K"/>
 <contactref element="20X_SENSOR" pad="17"/>
-<wire x1="7.607234375" y1="12.7" x2="190.5" y2="-1.27" width="0" layer="19" extent="1-1"/>
+<wire x1="7.607234375" y1="12.7" x2="210.82" y2="-1.27" width="0" layer="19" extent="1-1"/>
 </signal>
 <signal name="PHOTO9">
 <contactref element="D9" pad="K"/>
 <contactref element="20X_SENSOR" pad="4"/>
-<wire x1="129.545284375" y1="12.681946875" x2="208.28" y2="-3.81" width="0" layer="19" extent="1-1"/>
+<wire x1="193.04" y1="1.27" x2="129.545284375" y2="12.681946875" width="0" layer="19" extent="1-1"/>
 </signal>
 <signal name="PHOTO10">
 <contactref element="D10" pad="K"/>
 <contactref element="20X_SENSOR" pad="6"/>
-<wire x1="144.727390625" y1="12.669184375" x2="205.74" y2="-3.81" width="0" layer="19" extent="1-1"/>
+<wire x1="195.58" y1="1.27" x2="144.727390625" y2="12.669184375" width="0" layer="19" extent="1-1"/>
 </signal>
 <signal name="PHOTO11">
 <contactref element="D11" pad="K"/>
 <contactref element="20X_SENSOR" pad="8"/>
-<wire x1="160.007234375" y1="12.7" x2="203.2" y2="-3.81" width="0" layer="19" extent="1-1"/>
+<wire x1="198.12" y1="1.27" x2="160.007234375" y2="12.7" width="0" layer="19" extent="1-1"/>
 </signal>
 <signal name="PHOTO12">
 <contactref element="D12" pad="K"/>
 <contactref element="20X_SENSOR" pad="10"/>
-<wire x1="175.247234375" y1="12.7" x2="200.66" y2="-3.81" width="0" layer="19" extent="1-1"/>
+<wire x1="200.66" y1="1.27" x2="175.247234375" y2="12.7" width="0" layer="19" extent="1-1"/>
 </signal>
 <signal name="PHOTO13">
 <contactref element="D13" pad="K"/>
 <contactref element="20X_SENSOR" pad="12"/>
-<wire x1="198.12" y1="-3.81" x2="190.487234375" y2="12.7" width="0" layer="19" extent="1-1"/>
+<wire x1="203.2" y1="1.27" x2="190.487234375" y2="12.7" width="0" layer="19" extent="1-1"/>
 </signal>
 <signal name="PHOTO14">
 <contactref element="D14" pad="K"/>
 <contactref element="20X_SENSOR" pad="14"/>
-<wire x1="195.58" y1="-3.81" x2="205.727234375" y2="12.7" width="0" layer="19" extent="1-1"/>
+<wire x1="205.74" y1="1.27" x2="205.727234375" y2="12.7" width="0" layer="19" extent="1-1"/>
 </signal>
 <signal name="PHOTO15">
 <contactref element="D15" pad="K"/>
 <contactref element="20X_SENSOR" pad="16"/>
-<wire x1="193.04" y1="-3.81" x2="220.967234375" y2="12.7" width="0" layer="19" extent="1-1"/>
+<wire x1="208.28" y1="1.27" x2="220.967234375" y2="12.7" width="0" layer="19" extent="1-1"/>
 </signal>
 <signal name="N$2">
 <contactref element="R17" pad="1"/>
 <contactref element="IR" pad="A"/>
-<wire x1="15.24" y1="17.78" x2="12.7" y2="15.113" width="0" layer="19" extent="1-1"/>
+<wire x1="12.7" y1="15.113" x2="15.24" y2="22.86" width="0" layer="19" extent="1-1"/>
 </signal>
 <signal name="N$1">
@@
 <contactref element="R31" pad="1"/>
 <contactref element="IR14" pad="A"/>
-<wire x1="228.6" y1="17.78" x2="226.06" y2="15.113" width="0" layer="19" extent="1-1"/>
+<wire x1="226.06" y1="15.113" x2="228.6" y2="17.78" width="0" layer="19" extent="1-1"/>
+</signal>
+<signal name="+5V">
+<contactref element="20X_SENSOR" pad="2"/>
 </signal>
 </signals>
