File: Documents/EagleSchematics/THEBIGONE/THEBIGONE.brd (EAGLE design)
At the start: 99.1 x 160 mm, 32 parts, among them IC1 4067N, IC2 4067N, K1 612016235121, K2 612016235121, Q1 TIP120, Q2 TIP120, Q3 TIP120, Q4 TIP120, Q5 TIP120, Q6 TIP120

Commit message: Final
Final schematics
Connections:
- removed net PWM_SERVO4: K1.8
Changed lines of the file:
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@@
 <layer number="17" name="Pads" color="2" fill="1" visible="yes" active="yes"/>
 <layer number="18" name="Vias" color="2" fill="1" visible="yes" active="yes"/>
-<layer number="19" name="Unrouted" color="6" fill="1" visible="no" active="yes"/>
+<layer number="19" name="Unrouted" color="6" fill="1" visible="yes" active="yes"/>
 <layer number="20" name="Dimension" color="15" fill="1" visible="yes" active="yes"/>
 <layer number="21" name="tPlace" color="7" fill="1" visible="yes" active="yes"/>
@@
 <contactref element="K1" pad="6"/>
 </signal>
-<signal name="PWM_SERVO4">
-<contactref element="K1" pad="8"/>
-</signal>
 </signals>
