File: Documents/EagleSchematics/THEBIGONE/THEBIGONE.sch (EAGLE design)
At the start: 30 parts, among them Q1 TIP120, Q2 TIP120, Q3 TIP120, Q4 TIP120, Q5 TIP120

Commit message: Almost final version of schematics
Updated BigBoard with the new design
Parts:
- removed FROM_SENSOR_BOTTOM, FROM_SENSOR_TOP: 61202022021, Wuerth_Elektronik_eiCan_05_Box_Header_IDC_Connectors_1_2:61202022021
- removed JP3, JP4: (no value), SparkFun-Connectors:M03JST-PTH-VERT
- removed MULTIPLEX_1, MULTIPLEX_2: MUX-74HC4067SMD, SparkFun-AnalogIC:MUX-74HC4067SMD
- removed TO_MB_16PIN, TO_MB_16PIN1: 61201622021, Wuerth_Elektronik_eiCan_05_Box_Header_IDC_Connectors_1_2:61201622021
- added D6: 1N4004, diode:1N4004
- added FAN6: 22-23-2021, con-molex:22-23-2021
- added FROM_SENSORBOTTOM, FROM_SENSORTOP: 612020235121, Wuerth_Elektronik_eiCan_05_Box_Header_IDC_Connectors_1_2:612020235121
- added IC1, IC2: 4067N, 40xx:4067N
- added K1, K2: 612016235121, Wuerth_Elektronik_eiCan_05_Box_Header_IDC_Connectors_1_2:612016235121
- added Q6: TIP120, transistor-power:TIP120
- added R6: 2.2k, rcl:R-US_0204/7
Connections:
- removed net N$14: FROM_SENSOR_BOTTOM.19
- removed net N$15: FROM_SENSOR_BOTTOM.20
- new net N$16: Q6.B, R6.1
- new net N$17: D6.A, FAN6-2.S, Q6.C
- new net N$18: D6.C, FAN6-1.S
- new net N$19: FROM_SENSORTOP.19
- new net N$20: FROM_SENSORTOP.20
- new net PWM_LIFTFAN: K1.10, R6.2
- net +12V: now also K1.13; no longer TO_MB_16PIN.13
- net +5V: now also FROM_SENSORBOTTOM.2, FROM_SENSORTOP.2, K1.11; no longer FROM_SENSOR_BOTTOM.2, FROM_SENSOR_TOP.2, JP3.2, JP4.2, MULTIPLEX_1.VCC, MULTIPLEX_2.VCC, TO_MB_16PIN.11
- net DIG1: now also IC1A.A, K2.2; no longer MULTIPLEX_1.S0, TO_MB_16PIN1.2
- net DIG2: now also IC1A.B, K2.4; no longer MULTIPLEX_1.S1, TO_MB_16PIN1.4
- net DIG3: now also IC1A.C, K2.6; no longer MULTIPLEX_1.S2, TO_MB_16PIN1.6
- net DIG4: now also IC1A.D, K2.8; no longer MULTIPLEX_1.S3, TO_MB_16PIN1.8
- net DIG5: now also IC2A.A, K2.10; no longer MULTIPLEX_2.S0, TO_MB_16PIN1.10
- net DIG6: now also IC2A.B, K2.12; no longer MULTIPLEX_2.S1, TO_MB_16PIN1.12
- net DIG7: now also IC2A.C, K2.14; no longer MULTIPLEX_2.S2, TO_MB_16PIN1.14
- net DIG8: now also IC2A.D, K2.16; no longer MULTIPLEX_2.S3, TO_MB_16PIN1.16
- net GND: now also FROM_SENSORBOTTOM.1, FROM_SENSORTOP.1, IC1A.INH, IC2A.INH, K1.15, Q6.E; no longer FROM_SENSOR_BOTTOM.1, FROM_SENSOR_TOP.1, JP3.1, JP4.1, MULTIPLEX_1.EN, MULTIPLEX_1.GND, MULTIPLEX_2.EN, MULTIPLEX_2.GND, TO_MB_16PIN.15
- net MUX1: now also IC1A.X, K1.16; no longer MULTIPLEX_1.COM, TO_MB_16PIN.16
- net MUX2: now also IC2A.X, K1.14; no longer MULTIPLEX_2.COM, TO_MB_16PIN.14
- net N$26: now also FROM_SENSORBOTTOM.19; no longer FROM_SENSOR_TOP.19
- net N$27: now also FROM_SENSORBOTTOM.20; no longer FROM_SENSOR_TOP.20
- net PHOTO1: now also FROM_SENSORBOTTOM.3, IC1A.X0; no longer FROM_SENSOR_TOP.3, MULTIPLEX_1.CHAN0
- net PHOTO10: now also FROM_SENSORBOTTOM.6, IC1A.X9; no longer FROM_SENSOR_TOP.6, MULTIPLEX_1.CHAN9
- net PHOTO11: now also FROM_SENSORBOTTOM.8, IC1A.X10; no longer FROM_SENSOR_TOP.8, MULTIPLEX_1.CHAN10
- net PHOTO12: now also FROM_SENSORBOTTOM.10, IC1A.X11; no longer FROM_SENSOR_TOP.10, MULTIPLEX_1.CHAN11
- net PHOTO13: now also FROM_SENSORBOTTOM.12, IC1A.X12; no longer FROM_SENSOR_TOP.12, MULTIPLEX_1.CHAN12
- net PHOTO14: now also FROM_SENSORBOTTOM.14, IC1A.X13; no longer FROM_SENSOR_TOP.14, MULTIPLEX_1.CHAN13
- net PHOTO15: now also FROM_SENSORBOTTOM.16, IC1A.X14; no longer FROM_SENSOR_TOP.16, MULTIPLEX_1.CHAN14
- net PHOTO16: now also FROM_SENSORBOTTOM.18, IC1A.X15; no longer FROM_SENSOR_TOP.18, MULTIPLEX_1.CHAN15
- net PHOTO17: now also FROM_SENSORTOP.3, IC2A.X0; no longer FROM_SENSOR_BOTTOM.3, MULTIPLEX_2.CHAN0
- net PHOTO18: now also FROM_SENSORTOP.5, IC2A.X1; no longer FROM_SENSOR_BOTTOM.5, MULTIPLEX_2.CHAN1
- net PHOTO19: now also FROM_SENSORTOP.7, IC2A.X2; no longer FROM_SENSOR_BOTTOM.7, MULTIPLEX_2.CHAN2
- net PHOTO2: now also FROM_SENSORBOTTOM.5, IC1A.X1; no longer FROM_SENSOR_TOP.5, MULTIPLEX_1.CHAN1
- net PHOTO20: now also FROM_SENSORTOP.9, IC2A.X3; no longer FROM_SENSOR_BOTTOM.9, MULTIPLEX_2.CHAN3
- net PHOTO21: now also FROM_SENSORTOP.11, IC2A.X4; no longer FROM_SENSOR_BOTTOM.11, MULTIPLEX_2.CHAN4
- net PHOTO22: now also FROM_SENSORTOP.13, IC2A.X5; no longer FROM_SENSOR_BOTTOM.13, MULTIPLEX_2.CHAN5
- net PHOTO23: now also FROM_SENSORTOP.15, IC2A.X6; no longer FROM_SENSOR_BOTTOM.15, MULTIPLEX_2.CHAN6
- net PHOTO24: now also FROM_SENSORTOP.17, IC2A.X7; no longer FROM_SENSOR_BOTTOM.17, MULTIPLEX_2.CHAN7
- net PHOTO25: now also FROM_SENSORTOP.4, IC2A.X8; no longer FROM_SENSOR_BOTTOM.4, MULTIPLEX_2.CHAN8
- net PHOTO26: now also FROM_SENSORTOP.6, IC2A.X9; no longer FROM_SENSOR_BOTTOM.6, MULTIPLEX_2.CHAN9
- net PHOTO27: now also FROM_SENSORTOP.8, IC2A.X10; no longer FROM_SENSOR_BOTTOM.8, MULTIPLEX_2.CHAN10
- net PHOTO28: now also FROM_SENSORTOP.10, IC2A.X11; no longer FROM_SENSOR_BOTTOM.10, MULTIPLEX_2.CHAN11
- net PHOTO29: now also FROM_SENSORTOP.12, IC2A.X12; no longer FROM_SENSOR_BOTTOM.12, MULTIPLEX_2.CHAN12
- net PHOTO3: now also FROM_SENSORBOTTOM.7, IC1A.X2; no longer FROM_SENSOR_TOP.7, MULTIPLEX_1.CHAN2
- net PHOTO30: now also FROM_SENSORTOP.14, IC2A.X13; no longer FROM_SENSOR_BOTTOM.14, MULTIPLEX_2.CHAN13
- net PHOTO31: now also FROM_SENSORTOP.16, IC2A.X14; no longer FROM_SENSOR_BOTTOM.16, MULTIPLEX_2.CHAN14
- net PHOTO32: now also FROM_SENSORTOP.18, IC2A.X15; no longer FROM_SENSOR_BOTTOM.18, MULTIPLEX_2.CHAN15
- net PHOTO4: now also FROM_SENSORBOTTOM.9, IC1A.X3; no longer FROM_SENSOR_TOP.9, MULTIPLEX_1.CHAN3
- net PHOTO5: now also FROM_SENSORBOTTOM.11, IC1A.X4; no longer FROM_SENSOR_TOP.11, MULTIPLEX_1.CHAN4
- net PHOTO6: now also FROM_SENSORBOTTOM.13, IC1A.X5; no longer FROM_SENSOR_TOP.13, MULTIPLEX_1.CHAN5
- net PHOTO7: now also FROM_SENSORBOTTOM.15, IC1A.X6; no longer FROM_SENSOR_TOP.15, MULTIPLEX_1.CHAN6
- net PHOTO8: now also FROM_SENSORBOTTOM.17, IC1A.X7; no longer FROM_SENSOR_TOP.17, MULTIPLEX_1.CHAN7
- net PHOTO9: now also FROM_SENSORBOTTOM.4, IC1A.X8; no longer FROM_SENSOR_TOP.4, MULTIPLEX_1.CHAN8
- net PWM_FAN1: now also K1.1; no longer TO_MB_16PIN.1
- net PWM_FAN2: now also K1.3; no longer TO_MB_16PIN.3
- net PWM_FAN3: now also K1.5; no longer TO_MB_16PIN.5
- net PWM_FAN4: now also K1.7; no longer TO_MB_16PIN.7
- net PWM_FAN5: now also K1.9; no longer TO_MB_16PIN.9
- net PWM_SERVO1: now also K1.2; no longer TO_MB_16PIN.2
- net PWM_SERVO2: now also K1.4; no longer TO_MB_16PIN.4
- net PWM_SERVO3: now also K1.6; no longer JP3.3, TO_MB_16PIN.6
- net PWM_SERVO4: now also K1.8; no longer JP4.3, TO_MB_16PIN.8
Other:
- moved on the sheet: D1, D2, D3, D4, D5, FAN1-1, FAN1-2, FAN2-1, FAN2-2, FAN3-1, FAN3-2, FAN4-1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

Commit message: Final
Final schematics
Connections:
- removed net PWM_SERVO4: K1.8
Changed lines of the file:
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@@
 <segment>
 <wire x1="104.14" y1="99.06" x2="101.6" y2="99.06" width="0.1524" layer="91"/>
-<label x="104.14" y="99.06" size="1.27" layer="95" xref="yes"/>
 <pinref part="K1" gate="G$1" pin="6"/>
 </segment>
 </net>
-<net name="PWM_SERVO4" class="0">
-<segment>
-<wire x1="104.14" y1="93.98" x2="101.6" y2="93.98" width="0.1524" layer="91"/>
-<label x="104.14" y="93.98" size="1.016" layer="95" xref="yes"/>
-<pinref part="K1" gate="G$1" pin="8"/>
-</segment>
-</net>
